File: TABBx Lure 1.0.brd (EAGLE design)
At the start: 100 x 74.9 mm, 27 parts

Commit message: Route, throw in a LED... everyone likes LEDs
Parts:
- removed I2C: (no value), pinhead:1X04
- added I2CBUS01, I2CBUS02, I2CBUS03: (no value), pinhead:1X04
- added LED1: (no value), led:CHIPLED_1206
- added R0: (no value), adafruit:M1206
Connections:
- new net N$11: LED1.A, R0.2
- net 3.3V: now also R0.1
- net 5V: now also I2CBUS01.4, I2CBUS02.4, I2CBUS03.4; no longer I2C.4
- net GND: now also I2CBUS01.1, I2CBUS02.1, I2CBUS03.1, LED1.C; no longer I2C.1
- net SCL: now also I2CBUS01.3, I2CBUS02.3, I2CBUS03.3; no longer I2C.3
- net SDA: now also I2CBUS01.2, I2CBUS02.2, I2CBUS03.2; no longer I2C.2
Routing:
- net GND: track 0.00 -> 159.7 mm
- net GPIO0: track 0.00 -> 87.5 mm
- net UART2_RXD: track 0.00 -> 84.8 mm
- net GPIO2: track 0.00 -> 82.6 mm
- net UART2_TXD: track 0.00 -> 75.7 mm, vias 0 -> 2
- net UART1_RXD: track 0.00 -> 69.5 mm
- net GPIO1: track 0.00 -> 66.1 mm, vias 0 -> 1
- net GPIO5: track 0.00 -> 62.0 mm
- net UART1_TXD: track 0.00 -> 56.1 mm, vias 0 -> 1
- net SCL: track 0.00 -> 51.6 mm
- net 3.3V: track 0.00 -> 50.6 mm, vias 0 -> 2
- net GPIO7: track 0.00 -> 47.3 mm
- net 5V: track 0.00 -> 47.0 mm, vias 0 -> 2
- net GPIO3: track 0.00 -> 45.2 mm, vias 0 -> 1
- net GPIO4: track 0.00 -> 42.4 mm
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Other:
- board size 100 x 74.9 mm -> 99.1 x 73.7 mm
