File: TABBx Lure 1.0.sch (EAGLE design)
At the start: 27 parts

Commit message: Route, throw in a LED... everyone likes LEDs
Parts:
- added I2CBUS02, I2CBUS03: (no value), pinhead:PINHD-1X4
- added LED1: (no value), led:LEDCHIPLED_1206
- added R0: (no value), adafruit:R-US_M1206
- renumbered I2C to I2CBUS01
Connections:
- new net N$11: LED1.A, R0.2
- net 3.3V: now also R0.1
- net 5V: now also I2CBUS02.4, I2CBUS03.4
- net GND: now also I2CBUS02.1, I2CBUS03.1, LED1.C
- net SCL: now also I2CBUS02.3, I2CBUS03.3
- net SDA: now also I2CBUS02.2, I2CBUS03.2
